File: KiCad/FM_radio/FM_radio.kicad_pcb (KiCad board)
At the start: 2 copper layers, 33 x 48 mm, 77 parts, among them IC1 MCP73831T-2ACI_OT, IC2 SI4703-C19-GM, IC3 TPA741DR, IC4 TPA6111A2DR, J1 UJC-HP2-3-SMT-TR, J2 Conn_01x06_Pin, J3 SJ2-35853A-SMT-TR, U1 ATmega328P-A, Y1 ABS06N-32.768kHz-T

Commit message: Routing edit
Only few changes
Routing:
- net GND: track 30.0 -> 15.1 mm
Changed lines of the file:
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@@
 	)
 	(segment
+		(start 127.65 77.95)
+		(end 127.75 78.05)
+		(width 0.3)
+		(layer "F.Cu")
+		(net 5)
+	)
+	(segment
 		(start 128.65 75)
 		(end 128.4 75.25)
@@
 	)
 	(segment
+		(start 127.65 77.105)
+		(end 127.65 76)
+		(width 0.3)
+		(layer "F.Cu")
+		(net 5)
+	)
+	(segment
 		(start 128.15 77.105)
 		(end 128.15 76)
@@
 	)
 	(segment
+		(start 127.65 76)
+		(end 127.9 75.75)
+		(width 0.3)
+		(layer "F.Cu")
+		(net 5)
+	)
+	(segment
 		(start 127.15 74.1)
 		(end 127.15 74.395)
@@
 	)
 	(segment
-		(start 127.4 77.7)
-		(end 127.75 78.05)
-		(width 0.3)
-		(layer "B.Cu")
-		(net 5)
-	)
-	(segment
-		(start 127.1 76)
-		(end 127.1 74.2)
-		(width 0.3)
-		(layer "B.Cu")
-		(net 5)
-	)
-	(segment
-		(start 142.229354 74.309354)
-		(end 142.229354 75.530646)
-		(width 0.3)
-		(layer "B.Cu")
-		(net 5)
-	)
-	(segment
 		(start 139.6125 78.575)
 		(end 139.6125 78.6)
@@
 	)
 	(segment
-		(start 141.25 87.65)
-		(end 140.325 88.575)
-		(width 0.3)
-		(layer "B.Cu")
-		(net 5)
-	)
-	(segment
-		(start 136.75 74)
-		(end 136.75 75.51)
-		(width 0.3)
-		(layer "B.Cu")
-		(net 5)
-	)
-	(segment
 		(start 139.55 78.5125)
 		(end 139.6125 78.575)
@@
 	)
 	(segment
-		(start 127.4 76.3)
-		(end 127.1 76)
-		(width 0.3)
-		(layer "B.Cu")
-		(net 5)
-	)
-	(segment
-		(start 126.6 73.7)
-		(end 126.6 73.45)
-		(width 0.3)
-		(layer "B.Cu")
-		(net 5)
-	)
-	(segment
-		(start 133.699999 95.535158)
-		(end 131.599999 97.635158)
-		(width 0.3)
-		(layer "B.Cu")
-		(net 5)
-	)
-	(segment
 		(start 140.325 88.575)
 		(end 140.3 88.6)
@@
 	)
 	(segment
-		(start 129 73.85)
-		(end 129 73.35)
-		(width 0.3)
-		(layer "B.Cu")
-		(net 5)
-	)
-	(segment
-		(start 127.4 76.3)
-		(end 127.4 77.7)
-		(width 0.3)
-		(layer "B.Cu")
-		(net 5)
-	)
-	(segment
-		(start 141.25 87.3875)
-		(end 141.25 87.65)
-		(width 0.3)
-		(layer "B.Cu")
-		(net 5)
-	)
-	(segment
-		(start 128.4 74.45)
-		(end 129 73.85)
-		(width 0.3)
-		(layer "B.Cu")
-		(net 5)
-	)
-	(segment
-		(start 127.1 74.2)
-		(end 126.6 73.7)
-		(width 0.3)
-		(layer "B.Cu")
-		(net 5)
-	)
-	(segment
-		(start 131.599999 97.635158)
-		(end 131.599999 99.647658)
-		(width 0.3)
-		(layer "B.Cu")
-		(net 5)
-	)
-	(segment
 		(start 142.229354 75.530646)
 		(end 142.07 75.69)
@@
 	)
 	(segment
-		(start 128.4 75.25)
-		(end 128.4 74.45)
-		(width 0.3)
-		(layer "B.Cu")
-		(net 5)
-	)
-	(segment
 		(start 132.15 72.95)
 		(end 133.15 73.95)
@@
 	)
 	(segment
-		(start 143.15 78)
-		(end 143.15 80.35)
+		(start 143.15 80.35)
+		(end 143.8 81)
 		(width 0.3)
 		(layer "B.Cu")
@@
 	)
 	(segment
-		(start 137.95 74.7)
-		(end 137.95 75.666399)
+		(start 143.8 81)
+		(end 145.55 81)
 		(width 0.3)
 		(layer "B.Cu")
@@
 	)
 	(segment
-		(start 140.2 74.1)
-		(end 140.999354 74.899354)
+		(start 137.95 74.7)
+		(end 137.95 75.666399)
 		(width 0.3)
 		(layer "B.Cu")
@@
 	)
 	(segment
-		(start 151.292344 85.807656)
-		(end 151.292344 85.542227)
+		(start 138.5 74.15)
+		(end 138.55 74.1)
 		(width 0.3)
 		(layer "B.Cu")
@@
 	)
 	(segment
-		(start 145.55 81)
-		(end 146.3 81.75)
+		(start 141.5 77.1)
+		(end 142.25 77.1)
 		(width 0.3)
 		(layer "B.Cu")
@@
 	)
 	(segment
-		(start 138.5 74.15)
-		(end 137.95 74.7)
+		(start 140.999354 76.599354)
+		(end 141.5 77.1)
 		(width 0.3)
 		(layer "B.Cu")
@@
 	)
 	(segment
-		(start 138.55 74.1)
-		(end 140.2 74.1)
+		(start 147.75 88.4)
+		(end 149.6 88.4)
 		(width 0.3)
 		(layer "B.Cu")
@@
 	)
 	(segment
-		(start 143.15 80.35)
-		(end 143.8 81)
+		(start 146.3 81.75)
+		(end 146.3 86.95)
 		(width 0.3)
 		(layer "B.Cu")
@@
 	)
 	(segment
-		(start 141.45 77.05)
-		(end 141.5 77)
+		(start 143.15 78)
+		(end 143.15 80.35)
 		(width 0.3)
 		(layer "B.Cu")
@@
 	)
 	(segment
-		(start 149.6 88.4)
-		(end 150.05 87.95)
+		(start 146.3 86.95)
+		(end 147.75 88.4)
 		(width 0.3)
 		(layer "B.Cu")
@@
 	)
 	(segment
-		(start 140.999354 75.675753)
-		(end 140.999354 76.599354)
+		(start 145.55 81)
+		(end 146.3 81.75)
 		(width 0.3)
 		(layer "B.Cu")
@@
 	)
 	(segment
-		(start 146.3 81.75)
-		(end 146.3 86.95)
+		(start 140.999354 74.699354)
+		(end 140.999354 75.675753)
 		(width 0.3)
 		(layer "B.Cu")
@@
 	)
 	(segment
-		(start 150.05 87.95)
-		(end 150.05 87.05)
+		(start 149.6 88.4)
+		(end 150.05 87.95)
 		(width 0.3)
 		(layer "B.Cu")
@@
 	)
 	(segment
-		(start 143.8 81)
-		(end 145.55 81)
+		(start 138.55 74.1)
+		(end 140.4 74.1)
 		(width 0.3)
 		(layer "B.Cu")
@@
 	)
 	(segment
-		(start 146.3 86.95)
-		(end 147.75 88.4)
+		(start 138.5 74.15)
+		(end 137.95 74.7)
 		(width 0.3)
 		(layer "B.Cu")
@@
 	)
 	(segment
-		(start 137.945107 75.69)
-		(end 137.959354 75.675753)
+		(start 150.05 87.05)
+		(end 151.292344 85.807656)
 		(width 0.3)
 		(layer "B.Cu")
@@
 	)
 	(segment
-		(start 142.15 77)
-		(end 143.15 78)
+		(start 150.05 87.95)
+		(end 150.05 87.05)
 		(width 0.3)
 		(layer "B.Cu")
@@
 	)
 	(segment
-		(start 137.95 75.666399)
+		(start 137.945107 75.69)
 		(end 137.959354 75.675753)
 		(width 0.3)
@@
 	)
 	(segment
-		(start 141.5 77)
-		(end 142.15 77)
-		(width 0.3)
-		(layer "B.Cu")
-		(net 37)
-	)
-	(segment
-		(start 138.5 74.15)
-		(end 138.55 74.1)
+		(start 151.292344 85.807656)
+		(end 151.292344 85.542227)
 		(width 0.3)
 		(layer "B.Cu")
@@
 	)
 	(segment
-		(start 147.75 88.4)
-		(end 149.6 88.4)
+		(start 137.95 75.666399)
+		(end 137.959354 75.675753)
 		(width 0.3)
 		(layer "B.Cu")
@@
 	)
 	(segment
-		(start 140.999354 74.899354)
-		(end 140.999354 75.675753)
+		(start 140.4 74.1)
+		(end 140.999354 74.699354)
 		(width 0.3)
 		(layer "B.Cu")
@@
 	)
 	(segment
-		(start 140.999354 76.599354)
-		(end 141.45 77.05)
+		(start 142.25 77.1)
+		(end 143.15 78)
 		(width 0.3)
 		(layer "B.Cu")
@@
 	)
 	(segment
-		(start 150.05 87.05)
-		(end 151.292344 85.807656)
+		(start 140.999354 75.675753)
+		(end 140.999354 76.599354)
 		(width 0.3)
 		(layer "B.Cu")
